File: MiniB/minibergara.kicad_sch (KiCad schematic)
At the start: 12 parts, among them SW1 SW_Nidec_CAS-120A1, U1 TB6612_BREAKOUT, U2 LM7805_TO220

Commit message: boton y led puestos
hola
Parts:
- added D1: LED, LED_SMD:LED_0805_2012Metric, symbol Device:LED
- added J1: boton, Connector_PinHeader_2.54mm:PinHeader_1x02_P2.54mm_Vertical, symbol Connector:Conn_01x02_Pin
- added R1: R, Resistor_SMD:R_0805_2012Metric, symbol Device:R
Connections:
- net GND: now also D1.1 (K), J1.1 (Pin_1)
- net VCC: now also R1.2
- net d2: now reaches A1.5 (D2)
- net d2: now also J1.2 (Pin_2)
- new net: D1.2 (A), R1.1
Other:
- moved on the sheet: Entrada1, SW1
